Commit message: Test of adding IMU to xacro config

File: esa_proj/src/youbot/youbot_description/robots/youbot.urdf.xacro (robot description, xacro)
@@ -22,4 +22,5 @@
   <!-- sensors -->
   <xacro:include filename="$(find youbot_description)/urdf/sensors/hokuyo_urg04_laser.urdf.xacro"/>
+  <xacro:include filename="$(find youbot_description)/urdf/sensors/imu.xacro"/>
   <!-- Now we can start using the macros xacro:included above to define the actual youbot -->
   <!-- The first use of a macro.  This one was defined in base.urdf.xacro above.
@@ -45,3 +46,6 @@
     <origin xyz="0.3 0 -0.03" rpy="0 0 0"/>
   </xacro:hokuyo_urg04_laser>
+  <xacro:imu_sensor parent="base_link" xyz="0 0 0" rpy="0 0 0">
+    <origin xyz="0 0 0" rpy="0 0 0" />
+  </xacro:imu_sensor>
 </robot>
