Commit message: Update configs for Ubuntu 16.04

File: src/youbot/youbot_description/robots/youbot.urdf.xacro (robot description, xacro)
@@ -49,6 +49,3 @@
     <origin xyz="-0.3 0 -0.03" rpy="3.14 3.14 0"/>
   </xacro:hokuyo_urg04_laser>
-  <xacro:imu_sensor parent="base_link" xyz="0 0 0" rpy="0 0 0">
-    <origin xyz="0 0 0" rpy="0 0 0" />
-  </xacro:imu_sensor>
 </robot>

File: src/youbot/youbot_description/urdf/youbot_base/base.transmission.xacro (robot description, xacro)
@@ -6,5 +6,5 @@
 	<property name="wheel_mechanical_reduction" value="${624/35 * 80/18}" />
 	<property name="caster_mechanical_reduction" value="${624/35 * 80/18}" />
-	<property name="" value="0.360" />
+	<property name="_temp" value="0.360" />
 	<xacro:macro name="youbot_base_transmission">
 		<!-- front left wheel -->

Commit message: Geen idee

File: src/youbot/youbot_description/robots/youbot.urdf.xacro (robot description, xacro)
@@ -49,6 +49,3 @@
     <origin xyz="-0.3 0 -0.03" rpy="3.14 3.14 0"/>
   </xacro:hokuyo_urg04_laser>
-  <xacro:imu_sensor parent="base_link" xyz="0 0 0" rpy="0 0 0">
-    <origin xyz="0 0 0" rpy="0 0 0" />
-  </xacro:imu_sensor>
 </robot>
