Commit message: Fixed urdf warnings

File: src/youbot/youbot_description/robots/old/youbot.urdf.xacro (robot description, xacro)
@@ -1,4 +1,8 @@
 <?xml version="1.0"?>
-<robot xmlns:xacro="http://ros.org/wiki/xacro" name="youbot" >
+<robot xmlns:sensor="http://playerstage.sourceforge.net/gazebo/xmlschema/#sensor"
+       xmlns:controller="http://playerstage.sourceforge.net/gazebo/xmlschema/#controller"
+       xmlns:interface="http://playerstage.sourceforge.net/gazebo/xmlschema/#interface"
+       xmlns:xacro="http://playerstage.sourceforge.net/gazebo/xmlschema/#interface"
+       name="youbot" >
   <!-- The following xacro:included files set up definitions of parts of the robot body -->
   <!-- misc common stuff? -->
@@ -18,4 +22,5 @@
   <!-- sensors -->
   <xacro:include filename="$(find youbot_description)/urdf/sensors/hokuyo_urg04_laser.urdf.xacro"/>
+  <xacro:include filename="$(find youbot_description)/urdf/sensors/imu.xacro"/>
   <!-- Now we can start using the macros xacro:included above to define the actual youbot -->
   <!-- The first use of a macro.  This one was defined in base.urdf.xacro above.

File: src/youbot/youbot_description/urdf/youbot_base/base.transmission.xacro (robot description, xacro)
@@ -4,7 +4,7 @@
        xmlns:interface="http://playerstage.sourceforge.net/gazebo/xmlschema/#interface"
        xmlns:xacro="http://ros.org/wiki/xacro">
-	<property name="wheel_mechanical_reduction" value="${624/35 * 80/18}" />
-	<property name="caster_mechanical_reduction" value="${624/35 * 80/18}" />
-	<property name="empty" value="0.360" />
+	<xacro:property name="wheel_mechanical_reduction" value="${624/35 * 80/18}" />
+	<xacro:property name="caster_mechanical_reduction" value="${624/35 * 80/18}" />
+	<xacro:property name="empty" value="0.360" />
 	<xacro:macro name="youbot_base_transmission">
 		<!-- front left wheel -->

File: src/youbot/youbot_description/urdf/youbot_base/base.urdf.xacro (robot description, xacro)
@@ -8,28 +8,28 @@
   <xacro:include filename="$(find youbot_description)/urdf/youbot_base/base.transmission.xacro"/>
   <!-- simplified box collision geometry for base -->
-  <property name="base_size_x" value="0.570"/>
-  <property name="base_size_y" value="0.360"/>
-  <property name="base_size_z" value="0.100"/>
-  <property name="base_mass" value="22.0"/>
-  <property name="caster_offset_x" value="0.228"/>
-  <property name="caster_offset_y" value="0.158"/>
-  <property name="caster_offset_z" value="-0.034"/>
-  <property name="caster_mass" value="0.1"/>
-  <property name="wheel_offset_x" value="0.0"/>
-  <property name="wheel_offset_y" value="0.0"/>
-  <property name="wheel_offset_z" value="0.0"/>
-  <property name="wheel_mass" value="0.4"/>
-  <property name="wheel_radius" value="0.05"/>
-  <property name="wheel_length" value="0.005"/>
-  <property name="caster_joint_damping" value="1.0"/>
-  <property name="caster_joint_friction" value="1.0"/>
-  <property name="caster_joint_effort" value="30"/>
-  <property name="caster_joint_velocity" value="10"/>
-  <property name="caster_joint_safety_k_velocity" value="10.0"/>
-  <property name="wheel_joint_damping" value="1.0"/>
-  <property name="wheel_joint_friction" value="1.0"/>
-  <property name="wheel_joint_effort" value="30"/>
-  <property name="wheel_joint_velocity" value="10"/>
-  <property name="wheel_joint_safety_k_velocity" value="10.0"/>
+  <xacro:property name="base_size_x" value="0.570"/>
+  <xacro:property name="base_size_y" value="0.360"/>
+  <xacro:property name="base_size_z" value="0.100"/>
+  <xacro:property name="base_mass" value="22.0"/>
+  <xacro:property name="caster_offset_x" value="0.228"/>
+  <xacro:property name="caster_offset_y" value="0.158"/>
+  <xacro:property name="caster_offset_z" value="-0.034"/>
+  <xacro:property name="caster_mass" value="0.1"/>
+  <xacro:property name="wheel_offset_x" value="0.0"/>
+  <xacro:property name="wheel_offset_y" value="0.0"/>
+  <xacro:property name="wheel_offset_z" value="0.0"/>
+  <xacro:property name="wheel_mass" value="0.4"/>
+  <xacro:property name="wheel_radius" value="0.05"/>
+  <xacro:property name="wheel_length" value="0.005"/>
+  <xacro:property name="caster_joint_damping" value="1.0"/>
+  <xacro:property name="caster_joint_friction" value="1.0"/>
+  <xacro:property name="caster_joint_effort" value="30"/>
+  <xacro:property name="caster_joint_velocity" value="10"/>
+  <xacro:property name="caster_joint_safety_k_velocity" value="10.0"/>
+  <xacro:property name="wheel_joint_damping" value="1.0"/>
+  <xacro:property name="wheel_joint_friction" value="1.0"/>
+  <xacro:property name="wheel_joint_effort" value="30"/>
+  <xacro:property name="wheel_joint_velocity" value="10"/>
+  <xacro:property name="wheel_joint_safety_k_velocity" value="10.0"/>
   <xacro:macro name="youbot_base" params="name">
     <link name="${name}_footprint">

File: src/youbot/youbot_description/urdf/youbot_gripper/gripper.urdf.xacro (robot description, xacro)
@@ -10,5 +10,5 @@
 		<!-- joint between arm_7_link and sdh_palm_link -->
 		<joint name="${name}_palm_joint" type="fixed" >
-			<insert_block name="origin" />
+			<xacro:insert_block name="origin" />
 			<parent link="${parent}" />
 			<child link="${name}_palm_link" />
